File: Hardware/PianoBoard.brd (EAGLE design)
At the start: 185.4 x 80 mm, 159 parts

Commit message: placement update
Parts:
- moved OP20 125.6 mm to (97.8, 25.2), turned to 270 degrees
- moved OP18 92.9 mm to (70.7, 24.0), turned to 270 degrees
- moved OP19 88.1 mm to (59.3, 26.5), turned to 270 degrees
- moved OP21 75.9 mm to (24.9, 25.7), turned to 270 degrees
- moved R69 62.9 mm to (85.4, 8.66), turned to 90 degrees
- moved R65 47.3 mm to (87.2, 51.1)
- moved R64 47.3 mm to (87.2, 54.9)
- moved R66 47.3 mm to (87.2, 47.3)
- moved R67 47.3 mm to (87.2, 43.5)
- moved R68 47.3 mm to (87.2, 39.6)
- moved OP17 44.4 mm to (5.23, 37.6), turned to 270 degrees
- moved R9 27.4 mm to (40.2, 80.4)
- moved C3 26.9 mm to (-3.78, 49.7), turned to 90 degrees
- moved R70 26.9 mm to (80.9, 19.1), turned to 0 degrees
- moved OP4 26.2 mm to (45.3, 51.2)
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